Commit message: [Edit] joint limit

File: rhphumanoid_description/urdf/rhphumanoid.structure.larm.xacro (robot description, xacro)
@@ -35,7 +35,7 @@
     <parent link="l_sho_pitch_link"/>
     <child link="l_sho_roll_link"/>
-    <origin xyz="0.025420 0.037500 0.000000" rpy="0 0 0" />
+    <origin xyz="0.025420 0.037500 0.000000" rpy="${pi/2} 0 0" />
     <axis xyz="1 0 0" />
-    <limit effort="${45*9.80665/100}" velocity="${(pi/3)/0.18}" lower="${-pi*2/3}" upper="${pi*2/3}" />
+    <limit effort="${45*9.80665/100}" velocity="${(pi/3)/0.18}" lower="-1.8" upper="1.8" />
     <dynamics damping="0.1" friction="0.0" />
   </joint>
@@ -93,5 +93,5 @@
     <origin xyz="0.014000 -0.023610 -0.032830" rpy="0 0 0" />
     <axis xyz="0 1 0" />
-    <limit effort="${45*9.80665/100}" velocity="${(pi/3)/0.18}" lower="${-pi*2/3}" upper="${pi*2/3}" />
+    <limit effort="${45*9.80665/100}" velocity="${(pi/3)/0.18}" lower="${-pi/2}" upper="${pi*2/3}" />
     <dynamics damping="0.1" friction="0.0" />
   </joint>
@@ -121,5 +121,5 @@
     <origin xyz="0.015240 0.035670 -0.043170" rpy="0 0 0" />
     <axis xyz="1 0 0" />
-    <limit effort="${45*9.80665/100}" velocity="${(pi/3)/0.18}" lower="${-pi*2/3}" upper="${pi*2/3}" />
+    <limit effort="${45*9.80665/100}" velocity="${(pi/3)/0.18}" lower="-0.5" upper="0.2" />
     <dynamics damping="0.1" friction="0.0" />
   </joint>

File: rhphumanoid_description/urdf/rhphumanoid.structure.lleg.xacro (robot description, xacro)
@@ -37,5 +37,5 @@
     <origin xyz="-0.015830 0.000000 -0.035400" rpy="0 0 0" />
     <axis xyz="-1 0 0" />
-    <limit effort="${45*9.80665/100}" velocity="${(pi/3)/0.18}" lower="${-pi*2/3}" upper="${pi*2/3}" />
+    <limit effort="${45*9.80665/100}" velocity="${(pi/3)/0.18}" lower="-2.0" upper="2.0" />
     <dynamics damping="0.1" friction="0.0" />
   </joint>
@@ -65,5 +65,5 @@
     <origin xyz="0.016330 0.025420 0.000000" rpy="0 0 0" />
     <axis xyz="0 1 0" />
-    <limit effort="${45*9.80665/100}" velocity="${(pi/3)/0.18}" lower="${-pi*2/3}" upper="${pi*2/3}" />
+    <limit effort="${45*9.80665/100}" velocity="${(pi/3)/0.18}" lower="-0.55" upper="${pi*2/3}" />
     <dynamics damping="0.1" friction="0.0" />
   </joint>
@@ -93,5 +93,5 @@
     <origin xyz="0.000000 0.000000 -0.072100" rpy="0 0 0" />
     <axis xyz="0 1 0" />
-    <limit effort="${45*9.80665/100}" velocity="${(pi/3)/0.18}" lower="${-pi*2/3}" upper="${pi*2/3}" />
+    <limit effort="${45*9.80665/100}" velocity="${(pi/3)/0.18}" lower="${-pi*2/3}" upper="1.2" />
     <dynamics damping="0.1" friction="0.0" />
   </joint>
@@ -149,5 +149,5 @@
     <origin xyz="-0.016330 -0.025420 0.000000" rpy="0 0 0" />
     <axis xyz="1 0 0" />
-    <limit effort="${45*9.80665/100}" velocity="${(pi/3)/0.18}" lower="${-pi*2/3}" upper="${pi*2/3}" />
+    <limit effort="${45*9.80665/100}" velocity="${(pi/3)/0.18}" lower="-1.9" upper="1.9" />
     <dynamics damping="0.1" friction="0.0" />
   </joint>

File: rhphumanoid_description/urdf/rhphumanoid.structure.rarm.xacro (robot description, xacro)
@@ -35,7 +35,7 @@
     <parent link="r_sho_pitch_link"/>
     <child link="r_sho_roll_link"/>
-    <origin xyz="0.025420 -0.037500 0.000000" rpy="0 0 0" />
+    <origin xyz="0.025420 -0.037500 0.000000" rpy="${-pi/2} 0 0" />
     <axis xyz="1 0 0" />
-    <limit effort="${45*9.80665/100}" velocity="${(pi/3)/0.18}" lower="${-pi*2/3}" upper="${pi*2/3}" />
+    <limit effort="${45*9.80665/100}" velocity="${(pi/3)/0.18}" lower="-1.8" upper="1.8" />
     <dynamics damping="0.1" friction="0.0" />
   </joint>
@@ -93,5 +93,5 @@
     <origin xyz="0.014000 0.023610 -0.032830" rpy="0 0 0" />
     <axis xyz="0 -1 0" />
-    <limit effort="${45*9.80665/100}" velocity="${(pi/3)/0.18}" lower="${-pi*2/3}" upper="${pi*2/3}" />
+    <limit effort="${45*9.80665/100}" velocity="${(pi/3)/0.18}" lower="${-pi/2}" upper="${pi*2/3}" />
     <dynamics damping="0.1" friction="0.0" />
   </joint>
@@ -121,5 +121,5 @@
     <origin xyz="0.015240 -0.035670 -0.043170" rpy="0 0 0" />
     <axis xyz="1 0 0" />
-    <limit effort="${45*9.80665/100}" velocity="${(pi/3)/0.18}" lower="${-pi*2/3}" upper="${pi*2/3}" />
+    <limit effort="${45*9.80665/100}" velocity="${(pi/3)/0.18}" lower="-0.5" upper="0.2" />
     <dynamics damping="0.1" friction="0.0" />
   </joint>

File: rhphumanoid_description/urdf/rhphumanoid.structure.rleg.xacro (robot description, xacro)
@@ -37,5 +37,5 @@
     <origin xyz="-0.015830 0.000000 -0.035400" rpy="0 0 0" />
     <axis xyz="-1 0 0" />
-    <limit effort="${45*9.80665/100}" velocity="${(pi/3)/0.18}" lower="${-pi*2/3}" upper="${pi*2/3}" />
+    <limit effort="${45*9.80665/100}" velocity="${(pi/3)/0.18}" lower="-2" upper="2" />
     <dynamics damping="0.1" friction="0.0" />
   </joint>
@@ -65,5 +65,5 @@
     <origin xyz="0.016330 -0.025420 0.000000" rpy="0 0 0" />
     <axis xyz="0 -1 0" />
-    <limit effort="${45*9.80665/100}" velocity="${(pi/3)/0.18}" lower="${-pi*2/3}" upper="${pi*2/3}" />
+    <limit effort="${45*9.80665/100}" velocity="${(pi/3)/0.18}" lower="-0.5" upper="${pi*2/3}" />
     <dynamics damping="0.1" friction="0.0" />
   </joint>
@@ -93,5 +93,5 @@
     <origin xyz="0.000000 0.000000 -0.072100" rpy="0 0 0" />
     <axis xyz="0 -1 0" />
-    <limit effort="${45*9.80665/100}" velocity="${(pi/3)/0.18}" lower="${-pi*2/3}" upper="${pi*2/3}" />
+    <limit effort="${45*9.80665/100}" velocity="${(pi/3)/0.18}" lower="${-pi*2/3}" upper="1.2" />
     <dynamics damping="0.1" friction="0.0" />
   </joint>
@@ -149,5 +149,5 @@
     <origin xyz="-0.016330 0.025420 0.000000" rpy="0 0 0" />
     <axis xyz="1 0 0" />
-    <limit effort="${45*9.80665/100}" velocity="${(pi/3)/0.18}" lower="${-pi*2/3}" upper="${pi*2/3}" />
+    <limit effort="${45*9.80665/100}" velocity="${(pi/3)/0.18}" lower="-1.9" upper="1.9" />
     <dynamics damping="0.1" friction="0.0" />
   </joint>
