Commit message: [Modify] RHp Gazebo

File: rhphumanoid_description/urdf/rhphumanoid.gazebo.xacro (robot description, xacro)
@@ -1,5 +1,10 @@
 <?xml version="1.0"?>
 <robot xmlns:xacro="http://ros.org/wiki/xacro">
-  <xacro:macro name="robotis_op3_gazebo">
+  <xacro:macro name="rhphumanoid_gazebo" params="">
+    <gazebo>
+      <plugin filename="gz_ros2_control-system" name="gz_ros2_control::GazeboSimROS2ControlPlugin">
+        <parameters>$(find rhphumanoid_bringup)/config/rhphumanoid_controllers.yaml</parameters>
+      </plugin>
+    </gazebo>
     <gazebo reference="body_link">
       <mu1>0.2</mu1>
@@ -8,5 +13,4 @@
       <selfCollide>false</selfCollide>
     </gazebo>
-    <!-- left leg links -->
     <gazebo reference="l_hip_yaw_link">
       <mu1>0.2</mu1>
@@ -49,5 +53,4 @@
       <material>Gazebo/White</material>
     </gazebo>
-    <!-- right leg links -->
     <gazebo reference="r_hip_yaw_link">
       <mu1>0.2</mu1>
@@ -81,5 +84,4 @@
     </gazebo>
     <gazebo reference="r_ank_roll_link">
-      <mu1>9000</mu1>
       <kp>100000.0</kp>
       <kd>100.0</kd>
@@ -139,29 +141,4 @@
       <selfCollide>false</selfCollide>
     </gazebo>
-    <gazebo>
-      <plugin filename="gz-sim-joint-state-publisher-system" name = "gz::sim::systems::JointStatePublisher">
-        <topic>op3_gz_joint_states</topic>
-        <joint_name>r_sho_pitch</joint_name>
-        <joint_name>l_sho_pitch</joint_name>
-        <joint_name>r_sho_roll</joint_name>
-        <joint_name>l_sho_roll</joint_name>
-        <joint_name>r_el</joint_name>
-        <joint_name>l_el</joint_name>
-        <joint_name>r_hip_yaw</joint_name>
-        <joint_name>l_hip_yaw</joint_name>
-        <joint_name>r_hip_roll</joint_name>
-        <joint_name>l_hip_roll</joint_name>
-        <joint_name>r_hip_pitch</joint_name>
-        <joint_name>l_hip_pitch</joint_name>
-        <joint_name>r_knee</joint_name>
-        <joint_name>l_knee</joint_name>
-        <joint_name>r_ank_pitch</joint_name>
-        <joint_name>l_ank_pitch</joint_name>
-        <joint_name>r_ank_roll</joint_name>
-        <joint_name>l_ank_roll</joint_name>
-        <joint_name>head_pan</joint_name>
-        <joint_name>head_tilt</joint_name>
-      </plugin>
-    </gazebo>
     <gazebo reference="cam_gazebo_link">
       <sensor name='camera' type='camera'>
@@ -177,11 +154,11 @@
             <far>100.000000</far>
           </clip>
-          <camera_info_topic>camera_info</camera_info_topic>
-          <frame_id>/cam_gazebo_link</frame_id>
+          <camera_info_topic>camera/camera_info</camera_info_topic>
+          <frame_id>cam_gazebo_link</frame_id>
         </camera>
-        <alwaysOn>ture</alwaysOn>
+        <always_on>true</always_on>
         <visualize>true</visualize>
-        <update_rate>30.000000</update_rate>
-        <topic>image_raw</topic>
+        <update_rate>30.0</update_rate>
+        <topic>camera/image_raw</topic>
       </sensor>
     </gazebo>
@@ -191,5 +168,5 @@
         <imu>
           <enable_metrics>true</enable_metrics>
-          <frame_id>/cam_gazebo_link</frame_id>
+          <frame_id>body_link</frame_id>
         </imu>
         <always_on>true</always_on>

Commit message: [Modify] Gazebo Finish

File: rhphumanoid_description/urdf/rhphumanoid.gazebo.xacro (robot description, xacro)
@@ -10,5 +10,4 @@
       <mu1>0.2</mu1>
       <mu2>0.2</mu2>
-      <material>Gazebo/White</material>
       <selfCollide>false</selfCollide>
     </gazebo>
@@ -16,5 +15,4 @@
       <mu1>0.2</mu1>
       <mu2>0.2</mu2>
-      <material>Gazebo/White</material>
       <selfCollide>false</selfCollide>
     </gazebo>
@@ -22,5 +20,4 @@
       <mu1>0.2</mu1>
       <mu2>0.2</mu2>
-      <material>Gazebo/White</material>
       <selfCollide>false</selfCollide>
     </gazebo>
@@ -28,5 +25,4 @@
       <mu1>0.2</mu1>
       <mu2>0.2</mu2>
-      <material>Gazebo/White</material>
       <selfCollide>false</selfCollide>
     </gazebo>
@@ -34,5 +30,4 @@
       <mu1>0.2</mu1>
       <mu2>0.2</mu2>
-      <material>Gazebo/White</material>
       <selfCollide>false</selfCollide>
     </gazebo>
@@ -40,5 +35,4 @@
       <mu1>0.2</mu1>
       <mu2>0.2</mu2>
-      <material>Gazebo/White</material>
       <selfCollide>false</selfCollide>
     </gazebo>
@@ -51,10 +45,8 @@
       <maxVel>1.0</maxVel>
       <minDepth>0.001</minDepth>
-      <material>Gazebo/White</material>
     </gazebo>
     <gazebo reference="r_hip_yaw_link">
       <mu1>0.2</mu1>
       <mu2>0.2</mu2>
-      <material>Gazebo/White</material>
       <selfCollide>false</selfCollide>
     </gazebo>
@@ -62,5 +54,4 @@
       <mu1>0.2</mu1>
       <mu2>0.2</mu2>
-      <material>Gazebo/White</material>
       <selfCollide>false</selfCollide>
     </gazebo>
@@ -68,5 +59,4 @@
       <mu1>0.2</mu1>
       <mu2>0.2</mu2>
-      <material>Gazebo/White</material>
       <selfCollide>false</selfCollide>
     </gazebo>
@@ -74,5 +64,4 @@
       <mu1>0.2</mu1>
       <mu2>0.2</mu2>
-      <material>Gazebo/White</material>
       <selfCollide>false</selfCollide>
     </gazebo>
@@ -80,5 +69,4 @@
       <mu1>0.2</mu1>
       <mu2>0.2</mu2>
-      <material>Gazebo/White</material>
       <selfCollide>false</selfCollide>
     </gazebo>
@@ -91,10 +79,8 @@
       <maxVel>1.0</maxVel>
       <minDepth>0.001</minDepth>
-      <material>Gazebo/White</material>
     </gazebo>
     <gazebo reference="r_sho_pitch_link">
       <mu1>0.2</mu1>
       <mu2>0.2</mu2>
-      <material>Gazebo/White</material>
       <selfCollide>false</selfCollide>
     </gazebo>
@@ -102,5 +88,4 @@
       <mu1>0.2</mu1>
       <mu2>0.2</mu2>
-      <material>Gazebo/White</material>
       <selfCollide>false</selfCollide>
     </gazebo>
@@ -108,5 +93,4 @@
       <mu1>0.2</mu1>
       <mu2>0.2</mu2>
-      <material>Gazebo/White</material>
       <selfCollide>false</selfCollide>
     </gazebo>
@@ -114,5 +98,4 @@
       <mu1>0.2</mu1>
       <mu2>0.2</mu2>
-      <material>Gazebo/White</material>
       <selfCollide>false</selfCollide>
     </gazebo>
@@ -120,5 +103,4 @@
       <mu1>0.2</mu1>
       <mu2>0.2</mu2>
-      <material>Gazebo/White</material>
       <selfCollide>false</selfCollide>
     </gazebo>
@@ -126,5 +108,24 @@
       <mu1>0.2</mu1>
       <mu2>0.2</mu2>
-      <material>Gazebo/White</material>
+      <selfCollide>false</selfCollide>
+    </gazebo>
+    <gazebo reference="r_wst_link">
+      <mu1>0.2</mu1>
+      <mu2>0.2</mu2>
+      <selfCollide>false</selfCollide>
+    </gazebo>
+    <gazebo reference="r_grp_link">
+      <mu1>0.2</mu1>
+      <mu2>0.2</mu2>
+      <selfCollide>false</selfCollide>
+    </gazebo>
+    <gazebo reference="l_wst_link">
+      <mu1>0.2</mu1>
+      <mu2>0.2</mu2>
+      <selfCollide>false</selfCollide>
+    </gazebo>
+    <gazebo reference="l_grp_link">
+      <mu1>0.2</mu1>
+      <mu2>0.2</mu2>
       <selfCollide>false</selfCollide>
     </gazebo>
@@ -132,5 +133,4 @@
       <mu1>0.2</mu1>
       <mu2>0.2</mu2>
-      <material>Gazebo/White</material>
       <selfCollide>false</selfCollide>
     </gazebo>
@@ -138,5 +138,4 @@
       <mu1>0.2</mu1>
       <mu2>0.2</mu2>
-      <material>Gazebo/White</material>
       <selfCollide>false</selfCollide>
     </gazebo>
