Commit message: [Modify] Add head, Camera

File: rhphumanoid_description/urdf/rhphumanoid.inertia.xacro (robot description, xacro)
@@ -3,9 +3,9 @@
   <!-- body link -->
   <xacro:macro name="insert_inertia_body_link">
-    <origin xyz="0.00541350 -0.00007684 0.04633729" />
-    <mass value="0.82832100"/>
-    <inertia ixx="0.00247872" ixy="-0.00000075" ixz="-0.00003712"
-             iyy="0.00189302" iyz="-0.00000144"
-             izz="0.00175154" />
+    <origin xyz="0.00581692 -0.00007490 0.04314852" />
+    <mass value="0.91591488"/>
+    <inertia ixx="0.00296773" ixy="-0.00000063" ixz="-0.00002043"
+             iyy="0.00226577" iyz="-0.00000088"
+             izz="0.00194033" />
   </xacro:macro>
   <!-- right hip yaw link -->
@@ -187,17 +187,17 @@
   <!-- head yaw joint -->
   <xacro:macro name="insert_inertia_head_pan_link">
-    <origin xyz="0.00233 0.00000 0.00823" />
-    <mass value="0.01176"/>
-    <inertia ixx="0.00000397" ixy="0.0" ixz="-0.00000031"
-             iyy="0.00000165" iyz="0.0"
-             izz="0.00000387" />
+    <origin xyz="0.00416602 0.00168477 0.00322464" />
+    <mass value="0.02021093"/>
+    <inertia ixx="0.00000598" ixy="0.00000027" ixz="-0.00000079"
+             iyy="0.00000721" iyz="-0.00000044"
+             izz="0.00000469" />
   </xacro:macro>
   <!-- head pitch joint -->
   <xacro:macro name="insert_inertia_head_tilt_link">
-    <origin xyz="0.00230 -0.01863 0.02770" />
-    <mass value="0.13631"/>
-    <inertia ixx="0.00010612" ixy="0.00000011" ixz="-0.00000910"
-             iyy="0.00008721" iyz="0.00000084"
-             izz="0.00004529" />
+    <origin xyz="0.02426708 -0.01558055 0.02112161" />
+    <mass value="0.01056821"/>
+    <inertia ixx="0.00000420" ixy="-0.00000016" ixz="-0.00000123"
+             iyy="0.00000444" iyz="-0.00000015"
+             izz="0.00000394" />
   </xacro:macro>
 </robot>

File: rhphumanoid_description/urdf/rhphumanoid.structure.head.xacro (robot description, xacro)
@@ -7,5 +7,5 @@
     <parent link="${parent}"/>
     <child link="head_pan_link"/>
-    <origin xyz="-0.001 0.0 0.1365" rpy="0 0 0" />
+    <origin xyz="0.01841 0.0 0.1365" rpy="0 0 0" />
     <axis xyz="0 0 1" />
     <limit effort="${45*9.80665/100}" velocity="${(pi/3)/0.18}" lower="${-pi*2/3}" upper="${pi*2/3}" />
@@ -22,7 +22,7 @@
     </collision> -->
     <collision>
-      <origin xyz="0.003750 0.000000 0.015500" rpy="0 0 0"/>
+      <origin xyz="0.004670 0.000000 0.007000" rpy="0 0 0"/>
       <geometry>
-        <box size="0.032500 0.042000 0.031000"/>
+        <box size="0.049950 0.040000 0.053500"/>
       </geometry>
     </collision>
@@ -35,5 +35,5 @@
     <parent link="head_pan_link"/>
     <child link="head_tilt_link"/>
-    <origin xyz="0.010 0.019 0.0285" rpy="0 0 0" />
+    <origin xyz="0.01391 0.01538 0.01710" rpy="0 0 0" />
     <axis xyz="0 -1 0" />
     <limit effort="${45*9.80665/100}" velocity="${(pi/3)/0.18}" lower="${-pi*2/3}" upper="${pi*2/3}" />
@@ -50,7 +50,7 @@
     </collision> -->
     <collision>
-      <origin xyz="0.006000 -0.019000 0.027750" rpy="0 0 0"/>
+      <origin xyz="0.010980 -0.014970 0.021020" rpy="0 0 0"/>
       <geometry>
-        <box size="0.044500 0.094000 0.078000"/>
+        <box size="0.058010 0.040000 0.052110"/>
       </geometry>
     </collision>

File: rhphumanoid_description/urdf/rhphumanoid.urdf.xacro (robot description, xacro)
@@ -23,7 +23,7 @@
     </visual>
     <collision>
-      <origin xyz="0.0000 0.0000 0.0436" rpy="0 0 0"/>
+      <origin xyz="0.0000 0.0000 0.0407" rpy="0 0 0"/>
       <geometry>
-        <box size="0.1189 0.1321 0.1785"/>
+        <box size="0.1190 0.1321 0.1745"/>
       </geometry>
     </collision>

File: rhphumanoid_description/urdf/rhphumanoid.visuals.xacro (robot description, xacro)
@@ -238,5 +238,5 @@
     <origin xyz="0 0 0" rpy="0 0 0" />
     <geometry>
-      <mesh filename="package://rhphumanoid_description/meshes/la1.stl"  scale="0.001 0.001 0.001"/>
+      <mesh filename="package://rhphumanoid_description/meshes/head_pan.stl"  scale="0.001 0.001 0.001"/>
     </geometry>
     <material name="Grey">
@@ -248,5 +248,5 @@
     <origin xyz="0 0 0" rpy="0 0 0" />
     <geometry>
-      <mesh filename="package://rhphumanoid_description/meshes/la1.stl"  scale="0.001 0.001 0.001"/>
+      <mesh filename="package://rhphumanoid_description/meshes/head_tilt.stl"  scale="0.001 0.001 0.001"/>
     </geometry>
     <material name="Grey">
