Commit message: [Modify] Change head, Camera

File: rhphumanoid_description/urdf/rhphumanoid.structure.head.xacro (robot description, xacro)
@@ -61,10 +61,10 @@
   <!-- camera joint -->
   <joint name="cam" type="fixed">
-    <origin xyz="0.01425 -0.019 0.04975" rpy="${-pi*0.5} 0 ${-pi*0.5}"/>
+    <origin xyz="0.040 -0.015 0.027" rpy="${-pi*0.5} 0 ${-pi*0.5}"/>
     <parent link="head_tilt_link"/>
     <child link="cam_link"/>
   </joint>
   <joint name="cam_gazebo" type="fixed">
-    <origin xyz="0.01425 -0.019 0.04975" rpy="0 0 0"/>
+    <origin xyz="0.040 -0.015 0.027" rpy="0 0 0"/>
     <parent link="head_tilt_link"/>
     <child link="cam_gazebo_link"/>
