Commit message: [Modify] Add head structure

File: rhphumanoid_description/ros2_control/rhphumanoid.ros2_control.xacro (robot description, xacro)
@@ -124,4 +124,15 @@
         <state_interface name="velocity"/>
       </joint>
+      <!-- ==================== Head ==================== -->
+      <joint name="head_pan">
+        <command_interface name="position"/>
+        <state_interface name="position"/>
+        <state_interface name="velocity"/>
+      </joint>
+      <joint name="head_tilt">
+        <command_interface name="position"/>
+        <state_interface name="position"/>
+        <state_interface name="velocity"/>
+      </joint>
     </ros2_control>
   </xacro:macro>

File: rhphumanoid_description/urdf/rhphumanoid.inertia.xacro (robot description, xacro)
@@ -186,5 +186,5 @@
   </xacro:macro>
   <!-- head yaw joint -->
-  <!-- <xacro:macro name="insert_inertia_head_pan_link">
+  <xacro:macro name="insert_inertia_head_pan_link">
     <origin xyz="0.00233 0.00000 0.00823" />
     <mass value="0.01176"/>
@@ -192,7 +192,7 @@
              iyy="0.00000165" iyz="0.0"
              izz="0.00000387" />
-  </xacro:macro> -->
+  </xacro:macro>
   <!-- head pitch joint -->
-  <!-- <xacro:macro name="insert_inertia_head_tilt_link">
+  <xacro:macro name="insert_inertia_head_tilt_link">
     <origin xyz="0.00230 -0.01863 0.02770" />
     <mass value="0.13631"/>
@@ -200,4 +200,4 @@
              iyy="0.00008721" iyz="0.00000084"
              izz="0.00004529" />
-  </xacro:macro> -->
+  </xacro:macro>
 </robot>

File: rhphumanoid_description/urdf/rhphumanoid.structure.head.xacro (robot description, xacro)
@@ -2,5 +2,5 @@
 <robot xmlns:xacro="http://ros.org/wiki/xacro">
   <!-- head -->
-  <xacro:macro name="robotis_op3_head" params="parent">
+  <xacro:macro name="rhphumanoid_head" params="parent">
   <!-- head yaw joint -->
   <joint name="head_pan" type="revolute">
@@ -60,5 +60,5 @@
   </link>
   <!-- camera joint -->
-  <joint name="cam" type="fixed">
+  <!-- <joint name="cam" type="fixed">
     <origin xyz="0.01425 -0.019 0.04975" rpy="${-pi*0.5} 0 ${-pi*0.5}"/>
     <parent link="head_tilt_link"/>
@@ -69,11 +69,11 @@
     <parent link="head_tilt_link"/>
     <child link="cam_gazebo_link"/>
-  </joint>
+  </joint> -->
   <!-- camera link -->
-  <link name="cam_link">
-  </link>
+  <!-- <link name="cam_link">
+  </link> -->
   <!-- camera link -->
-  <link name="cam_gazebo_link">
-  </link>
+  <!-- <link name="cam_gazebo_link">
+  </link> -->
   </xacro:macro>
 </robot>

File: rhphumanoid_description/urdf/rhphumanoid.urdf.xacro (robot description, xacro)
@@ -8,5 +8,5 @@
   <xacro:include filename="$(find rhphumanoid_description)/urdf/rhphumanoid.structure.rleg.xacro" />
   <xacro:include filename="$(find rhphumanoid_description)/urdf/rhphumanoid.structure.lleg.xacro" />
-  <!-- <xacro:include filename="$(find rhphumanoid_description)/urdf/rhphumanoid.structure.head.xacro" /> -->
+  <xacro:include filename="$(find rhphumanoid_description)/urdf/rhphumanoid.structure.head.xacro" />
   <!-- <xacro:include filename="$(find rhphumanoid_description)/urdf/rhphumanoid.ros2.gazebo.xacro" /> -->
   <xacro:include filename="$(find rhphumanoid_description)/ros2_control/rhphumanoid.ros2_control.xacro" />
@@ -37,5 +37,5 @@
   <xacro:rhphumanoid_ros2_control name="RHPHumanoid" use_gazebo="$(arg use_gazebo)" />
   <!-- head links -->
-  <!-- <xacro:rhphumanoid_head parent="body_link" />   -->
+  <xacro:rhphumanoid_head parent="body_link" />
   <xacro:if value="$(arg use_gazebo)">
     <xacro:include filename="$(find rhphumanoid_description)/gazebo/rhphumanoid.gazebo.xacro" />

File: rhphumanoid_description/urdf/rhphumanoid.visuals.xacro (robot description, xacro)
@@ -235,22 +235,22 @@
   </xacro:macro>
   <!-- head yaw joint -->
-  <!-- <xacro:macro name="insert_mesh_head_pan_link">
-    <origin xyz="0 0 0" rpy="0 0 0" />
-    <geometry>
-      <mesh filename="package://rhphumanoid_description/meshes/h1.stl"  scale="0.001 0.001 0.001"/>
+  <xacro:macro name="insert_mesh_head_pan_link">
+    <origin xyz="0 0 0" rpy="0 0 0" />
+    <geometry>
+      <mesh filename="package://rhphumanoid_description/meshes/la1.stl"  scale="0.001 0.001 0.001"/>
     </geometry>
     <material name="Grey">
       <color rgba="0.60 0.60 0.60 1.0"/>
     </material>
-  </xacro:macro> -->
+  </xacro:macro>
   <!-- head yaw joint -->
-  <!-- <xacro:macro name="insert_mesh_head_tilt_link">
-    <origin xyz="0 0 0" rpy="0 0 0" />
-    <geometry>
-      <mesh filename="package://rhphumanoid_description/meshes/h2.stl"  scale="0.001 0.001 0.001"/>
+  <xacro:macro name="insert_mesh_head_tilt_link">
+    <origin xyz="0 0 0" rpy="0 0 0" />
+    <geometry>
+      <mesh filename="package://rhphumanoid_description/meshes/la1.stl"  scale="0.001 0.001 0.001"/>
     </geometry>
     <material name="Grey">
       <color rgba="0.60 0.60 0.60 1.0"/>
     </material>
-  </xacro:macro> -->
+  </xacro:macro>
 </robot>

Commit message: [Modify] Fix Gazebo sim performance and migrate to ros_gz packages

File: rhphumanoid_description/ros2_control/rhphumanoid.ros2_control.xacro (robot description, xacro)
@@ -5,5 +5,5 @@
       <hardware>
         <xacro:if value="${use_gazebo}">
-          <plugin>ign_ros2_control/IgnitionSystem</plugin>
+          <plugin>gz_ros2_control/GazeboSimSystem</plugin>
         </xacro:if>
         <xacro:unless value="${use_gazebo}">

File: rhphumanoid_description/urdf/rhphumanoid.gazebo.xacro (robot description, xacro)
@@ -3,5 +3,5 @@
   <xacro:macro name="rhphumanoid_gazebo" params="">
     <gazebo>
-      <plugin filename="gz_ros2_control-system" name="ign_ros2_control::GazeboSimROS2ControlPlugin">
+      <plugin filename="gz_ros2_control-system" name="gz_ros2_control::GazeboSimROS2ControlPlugin">
         <parameters>$(find rhphumanoid_bringup)/config/rhphumanoid_controllers.yaml</parameters>
       </plugin>
@@ -142,5 +142,5 @@
     <gazebo reference="cam_gazebo_link">
       <sensor name='camera' type='camera'>
-        <ign_frame_id>cam_gazebo_link</ign_frame_id>
+        <gz_frame_id>cam_gazebo_link</gz_frame_id>
         <camera name='__default__'>
           <horizontal_fov>1.012300</horizontal_fov>
@@ -164,5 +164,5 @@
     <gazebo reference="body_link">
       <sensor name="imu" type="imu">
-        <ign_frame_id>body_link</ign_frame_id>
+        <gz_frame_id>body_link</gz_frame_id>
         <imu>
           <enable_metrics>true</enable_metrics>

File: rhphumanoid_description/urdf/rhphumanoid.structure.larm.xacro (robot description, xacro)
@@ -19,12 +19,9 @@
     </visual>
     <collision>
-      <xacro:insert_mesh_l_sho_pitch_link />
+      <origin xyz="-0.0001 0.0220 0.0000" rpy="0 0 0"/>
+      <geometry>
+        <box size="0.0510 0.0511 0.0300"/>
+      </geometry>
     </collision>
-    <!-- <collision>
-      <origin xyz="0 0 0" rpy="0 0 0"/>
-      <geometry>
-        <box size="0 0 0"/>
-      </geometry>
-    </collision> -->
     <inertial>
       <xacro:insert_inertia_l_sho_pitch_link />
@@ -47,12 +44,9 @@
     </visual>
     <collision>
-      <xacro:insert_mesh_l_sho_roll_link />
+      <origin xyz="-0.0252 0.0051 -0.0259" rpy="0 0 0"/>
+      <geometry>
+        <box size="0.0572 0.0401 0.0716"/>
+      </geometry>
     </collision>
-    <!-- <collision>
-      <origin xyz="0 0 0" rpy="0 0 0"/>
-      <geometry>
-        <box size="0 0 0"/>
-      </geometry>
-    </collision> -->
     <inertial>
       <xacro:insert_inertia_l_sho_roll_link />
@@ -75,12 +69,9 @@
     </visual>
     <collision>
-      <xacro:insert_mesh_l_el_link />
+      <origin xyz="0.0044 0.0000 -0.0196" rpy="0 0 0"/>
+      <geometry>
+        <box size="0.0391 0.0572 0.0465"/>
+      </geometry>
     </collision>
-    <!-- <collision>
-      <origin xyz="0 0 0" rpy="0 0 0"/>
-      <geometry>
-        <box size="0 0 0"/>
-      </geometry>
-    </collision> -->
     <inertial>
       <xacro:insert_inertia_l_el_link />
@@ -103,12 +94,9 @@
     </visual>
     <collision>
-      <xacro:insert_mesh_l_wst_link />
+      <origin xyz="-0.0102 0.0228 -0.0520" rpy="0 0 0"/>
+      <geometry>
+        <box size="0.0536 0.0564 0.1241"/>
+      </geometry>
     </collision>
-    <!-- <collision>
-      <origin xyz="0 0 0" rpy="0 0 0"/>
-      <geometry>
-        <box size="0 0 0"/>
-      </geometry>
-    </collision> -->
     <inertial>
       <xacro:insert_inertia_l_wst_link />
@@ -131,12 +119,9 @@
     </visual>
     <collision>
-      <xacro:insert_mesh_l_grp_link />
+      <origin xyz="-0.0252 0.0070 -0.0305" rpy="0 0 0"/>
+      <geometry>
+        <box size="0.0572 0.0340 0.0810"/>
+      </geometry>
     </collision>
-    <!-- <collision>
-      <origin xyz="0 0 0" rpy="0 0 0"/>
-      <geometry>
-        <box size="0 0 0"/>
-      </geometry>
-    </collision> -->
     <inertial>
       <xacro:insert_inertia_l_grp_link />

File: rhphumanoid_description/urdf/rhphumanoid.structure.lleg.xacro (robot description, xacro)
@@ -19,12 +19,9 @@
     </visual>
     <collision>
-      <xacro:insert_mesh_l_hip_yaw_link />
+      <origin xyz="0.0000 0.0000 -0.0209" rpy="0 0 0"/>
+      <geometry>
+        <box size="0.0389 0.0300 0.0490"/>
+      </geometry>
     </collision>
-    <!-- <collision>
-      <origin xyz="0 0 0" rpy="0 0 0"/>
-      <geometry>
-        <box size="0 0 0"/>
-      </geometry>
-    </collision> -->
     <inertial>
       <xacro:insert_inertia_l_hip_yaw_link />
@@ -47,12 +44,9 @@
     </visual>
     <collision>
-      <xacro:insert_mesh_l_hip_roll_link />
+      <origin xyz="-0.0086 -0.0001 -0.0125" rpy="0 0 0"/>
+      <geometry>
+        <box size="0.0848 0.0510 0.0451"/>
+      </geometry>
     </collision>
-    <!-- <collision>
-      <origin xyz="0 0 0" rpy="0 0 0"/>
-      <geometry>
-        <box size="0 0 0"/>
-      </geometry>
-    </collision> -->
     <inertial>
       <xacro:insert_inertia_l_hip_roll_link />
@@ -75,12 +69,9 @@
     </visual>
     <collision>
-      <xacro:insert_mesh_l_hip_pitch_link />
+      <origin xyz="0.0000 -0.0247 -0.0360" rpy="0 0 0"/>
+      <geometry>
+        <box size="0.0201 0.0543 0.0921"/>
+      </geometry>
     </collision>
-    <!-- <collision>
-      <origin xyz="0 0 0" rpy="0 0 0"/>
-      <geometry>
-        <box size="0 0 0"/>
-      </geometry>
-    </collision> -->
     <inertial>
       <xacro:insert_inertia_l_hip_pitch_link />
@@ -103,12 +94,9 @@
     </visual>
     <collision>
-      <xacro:insert_mesh_l_knee_link />
+      <origin xyz="0.0000 -0.0247 -0.0360" rpy="0 0 0"/>
+      <geometry>
+        <box size="0.0200 0.0543 0.0920"/>
+      </geometry>
     </collision>
-    <!-- <collision>
-      <origin xyz="0 0 0" rpy="0 0 0"/>
-      <geometry>
-        <box size="0 0 0"/>
-      </geometry>
-    </collision> -->
     <inertial>
       <xacro:insert_inertia_l_knee_link />
@@ -131,12 +119,9 @@
     </visual>
     <collision>
-      <xacro:insert_mesh_l_ank_pitch_link />
+      <origin xyz="-0.0249 -0.0255 0.0133" rpy="0 0 0"/>
+      <geometry>
+        <box size="0.0848 0.0510 0.0466"/>
+      </geometry>
     </collision>
-    <!-- <collision>
-      <origin xyz="0 0 0" rpy="0 0 0"/>
-      <geometry>
-        <box size="0 0 0"/>
-      </geometry>
-    </collision> -->
     <inertial>
       <xacro:insert_inertia_l_ank_pitch_link />
@@ -159,12 +144,9 @@
     </visual>
     <collision>
-      <xacro:insert_mesh_l_ank_roll_link />
+      <origin xyz="0.0172 0.0080 -0.0140" rpy="0 0 0"/>
+      <geometry>
+        <box size="0.1000 0.0800 0.0480"/>
+      </geometry>
     </collision>
-    <!-- <collision>
-      <origin xyz="0 0 0" rpy="0 0 0"/>
-      <geometry>
-        <box size="0 0 0"/>
-      </geometry>
-    </collision> -->
     <inertial>
       <xacro:insert_inertia_l_ank_roll_link />

File: rhphumanoid_description/urdf/rhphumanoid.structure.rarm.xacro (robot description, xacro)
@@ -19,12 +19,9 @@
     </visual>
     <collision>
-      <xacro:insert_mesh_r_sho_pitch_link />
+      <origin xyz="-0.0001 -0.0220 0.0000" rpy="0 0 0"/>
+      <geometry>
+        <box size="0.0510 0.0511 0.0300"/>
+      </geometry>
     </collision>
-    <!-- <collision>
-      <origin xyz="0 0 0" rpy="0 0 0"/>
-      <geometry>
-        <box size="0 0 0"/>
-      </geometry>
-    </collision> -->
     <inertial>
       <xacro:insert_inertia_r_sho_pitch_link />
@@ -47,12 +44,9 @@
     </visual>
     <collision>
-      <xacro:insert_mesh_r_sho_roll_link />
+      <origin xyz="-0.0252 -0.0051 -0.0259" rpy="0 0 0"/>
+      <geometry>
+        <box size="0.0572 0.0401 0.0716"/>
+      </geometry>
     </collision>
-    <!-- <collision>
-      <origin xyz="0 0 0" rpy="0 0 0"/>
-      <geometry>
-        <box size="0 0 0"/>
-      </geometry>
-    </collision> -->
     <inertial>
       <xacro:insert_inertia_r_sho_roll_link />
@@ -75,12 +69,9 @@
     </visual>
     <collision>
-      <xacro:insert_mesh_r_el_link />
+      <origin xyz="0.0044 0.0000 -0.0196" rpy="0 0 0"/>
+      <geometry>
+        <box size="0.0391 0.0572 0.0465"/>
+      </geometry>
     </collision>
-    <!-- <collision>
-      <origin xyz="0 0 0" rpy="0 0 0"/>
-      <geometry>
-        <box size="0 0 0"/>
-      </geometry>
-    </collision> -->
     <inertial>
       <xacro:insert_inertia_r_el_link />
@@ -103,12 +94,9 @@
     </visual>
     <collision>
-      <xacro:insert_mesh_r_wst_link />
+      <origin xyz="-0.0102 -0.0228 -0.0520" rpy="0 0 0"/>
+      <geometry>
+        <box size="0.0536 0.0564 0.1241"/>
+      </geometry>
     </collision>
-    <!-- <collision>
-      <origin xyz="0 0 0" rpy="0 0 0"/>
-      <geometry>
-        <box size="0 0 0"/>
-      </geometry>
-    </collision> -->
     <inertial>
       <xacro:insert_inertia_r_wst_link />
@@ -131,12 +119,9 @@
     </visual>
     <collision>
-      <xacro:insert_mesh_r_grp_link />
+      <origin xyz="-0.0252 -0.0070 -0.0305" rpy="0 0 0"/>
+      <geometry>
+        <box size="0.0572 0.0340 0.0810"/>
+      </geometry>
     </collision>
-    <!-- <collision>
-      <origin xyz="0 0 0" rpy="0 0 0"/>
-      <geometry>
-        <box size="0 0 0"/>
-      </geometry>
-    </collision> -->
     <inertial>
       <xacro:insert_inertia_r_grp_link />

File: rhphumanoid_description/urdf/rhphumanoid.structure.rleg.xacro (robot description, xacro)
@@ -19,12 +19,9 @@
     </visual>
     <collision>
-      <xacro:insert_mesh_r_hip_yaw_link />
+      <origin xyz="0.0000 0.0000 -0.0209" rpy="0 0 0"/>
+      <geometry>
+        <box size="0.0389 0.0300 0.0490"/>
+      </geometry>
     </collision>
-    <!-- <collision>
-      <origin xyz="0 0 0" rpy="0 0 0"/>
-      <geometry>
-        <box size="0 0 0"/>
-      </geometry>
-    </collision> -->
     <inertial>
       <xacro:insert_inertia_r_hip_yaw_link />
@@ -47,12 +44,9 @@
     </visual>
     <collision>
-      <xacro:insert_mesh_r_hip_roll_link />
+      <origin xyz="-0.0086 0.0001 -0.0125" rpy="0 0 0"/>
+      <geometry>
+        <box size="0.0848 0.0510 0.0451"/>
+      </geometry>
     </collision>
-    <!-- <collision>
-      <origin xyz="0 0 0" rpy="0 0 0"/>
-      <geometry>
-        <box size="0 0 0"/>
-      </geometry>
-    </collision> -->
     <inertial>
       <xacro:insert_inertia_r_hip_roll_link />
@@ -75,12 +69,9 @@
     </visual>
     <collision>
-      <xacro:insert_mesh_r_hip_pitch_link />
+      <origin xyz="0.0000 0.0247 -0.0360" rpy="0 0 0"/>
+      <geometry>
+        <box size="0.0201 0.0543 0.0921"/>
+      </geometry>
     </collision>
-    <!-- <collision>
-      <origin xyz="0 0 0" rpy="0 0 0"/>
-      <geometry>
-        <box size="0 0 0"/>
-      </geometry>
-    </collision> -->
     <inertial>
       <xacro:insert_inertia_r_hip_pitch_link />
@@ -103,12 +94,9 @@
     </visual>
     <collision>
-      <xacro:insert_mesh_r_knee_link />
+      <origin xyz="0.0000 0.0247 -0.0360" rpy="0 0 0"/>
+      <geometry>
+        <box size="0.0200 0.0543 0.0920"/>
+      </geometry>
     </collision>
-    <!-- <collision>
-      <origin xyz="0 0 0" rpy="0 0 0"/>
-      <geometry>
-        <box size="0 0 0"/>
-      </geometry>
-    </collision> -->
     <inertial>
       <xacro:insert_inertia_r_knee_link />
@@ -131,12 +119,9 @@
     </visual>
     <collision>
-      <xacro:insert_mesh_r_ank_pitch_link />
+      <origin xyz="-0.0249 0.0255 0.0133" rpy="0 0 0"/>
+      <geometry>
+        <box size="0.0848 0.0510 0.0466"/>
+      </geometry>
     </collision>
-    <!-- <collision>
-      <origin xyz="0 0 0" rpy="0 0 0"/>
-      <geometry>
-        <box size="0 0 0"/>
-      </geometry>
-    </collision> -->
     <inertial>
       <xacro:insert_inertia_r_ank_pitch_link />
@@ -159,12 +144,9 @@
     </visual>
     <collision>
-      <xacro:insert_mesh_r_ank_roll_link />
+      <origin xyz="0.0181 -0.0080 -0.0140" rpy="0 0 0"/>
+      <geometry>
+        <box size="0.1000 0.0800 0.0480"/>
+      </geometry>
     </collision>
-    <!-- <collision>
-      <origin xyz="0 0 0" rpy="0 0 0"/>
-      <geometry>
-        <box size="0 0 0"/>
-      </geometry>
-    </collision> -->
     <inertial>
       <xacro:insert_inertia_r_ank_roll_link />

File: rhphumanoid_description/urdf/rhphumanoid.urdf.xacro (robot description, xacro)
@@ -17,12 +17,9 @@
     </visual>
     <collision>
-      <xacro:insert_mesh_body_link />
+      <origin xyz="0.0000 0.0000 0.0436" rpy="0 0 0"/>
+      <geometry>
+        <box size="0.1189 0.1321 0.1785"/>
+      </geometry>
     </collision>
-    <!-- <collision>
-      <origin xyz="0 0 0" rpy="0 0 0"/>
-      <geometry>
-        <box size="0 0 0"/>
-      </geometry>
-    </collision> -->
     <inertial>
       <xacro:insert_inertia_body_link />
