Commit message: [Add] PWM head hardware plugin and head controller package

File: rhphumanoid_description/ros2_control/rhphumanoid.ros2_control.xacro (robot description, xacro)
@@ -2,161 +2,346 @@
 <robot xmlns:xacro="http://www.ros.org/wiki/xacro">
   <xacro:macro name="rhphumanoid_ros2_control" params="name use_gazebo:=^|false">
-    <ros2_control name="${name}" type="system">
-      <hardware>
-        <xacro:if value="${use_gazebo}">
+    <!-- ============================================================== -->
+    <!-- GAZEBO SIMULATION: single system with all 24 joints            -->
+    <!-- ============================================================== -->
+    <xacro:if value="${use_gazebo}">
+      <ros2_control name="${name}" type="system">
+        <hardware>
           <plugin>gz_ros2_control/GazeboSimSystem</plugin>
-        </xacro:if>
-        <xacro:unless value="${use_gazebo}">
+        </hardware>
+        <!-- Left Arm -->
+        <joint name="l_sho_pitch">
+          <command_interface name="position"/>
+          <state_interface name="position">
+            <param name="initial_value">0.15</param>
+          </state_interface>
+        </joint>
+        <joint name="l_sho_roll">
+          <command_interface name="position"/>
+          <state_interface name="position">
+            <param name="initial_value">-1.45</param>
+          </state_interface>
+        </joint>
+        <joint name="l_el">
+          <command_interface name="position"/>
+          <state_interface name="position">
+            <param name="initial_value">0.0</param>
+          </state_interface>
+        </joint>
+        <joint name="l_wst">
+          <command_interface name="position"/>
+          <state_interface name="position">
+            <param name="initial_value">-0.5</param>
+          </state_interface>
+        </joint>
+        <joint name="l_grp">
+          <command_interface name="position"/>
+          <state_interface name="position">
+            <param name="initial_value">0.0</param>
+          </state_interface>
+        </joint>
+        <!-- Right Arm -->
+        <joint name="r_sho_pitch">
+          <command_interface name="position"/>
+          <state_interface name="position">
+            <param name="initial_value">-0.15</param>
+          </state_interface>
+        </joint>
+        <joint name="r_sho_roll">
+          <command_interface name="position"/>
+          <state_interface name="position">
+            <param name="initial_value">1.45</param>
+          </state_interface>
+        </joint>
+        <joint name="r_el">
+          <command_interface name="position"/>
+          <state_interface name="position">
+            <param name="initial_value">0.0</param>
+          </state_interface>
+        </joint>
+        <joint name="r_wst">
+          <command_interface name="position"/>
+          <state_interface name="position">
+            <param name="initial_value">0.5</param>
+          </state_interface>
+        </joint>
+        <joint name="r_grp">
+          <command_interface name="position"/>
+          <state_interface name="position">
+            <param name="initial_value">0.0</param>
+          </state_interface>
+        </joint>
+        <!-- Left Leg -->
+        <joint name="l_hip_yaw">
+          <command_interface name="position"/>
+          <state_interface name="position">
+            <param name="initial_value">0.0</param>
+          </state_interface>
+        </joint>
+        <joint name="l_hip_roll">
+          <command_interface name="position"/>
+          <state_interface name="position">
+            <param name="initial_value">0.0</param>
+          </state_interface>
+        </joint>
+        <joint name="l_hip_pitch">
+          <command_interface name="position"/>
+          <state_interface name="position">
+            <param name="initial_value">0.0</param>
+          </state_interface>
+        </joint>
+        <joint name="l_knee">
+          <command_interface name="position"/>
+          <state_interface name="position">
+            <param name="initial_value">0.0</param>
+          </state_interface>
+        </joint>
+        <joint name="l_ank_pitch">
+          <command_interface name="position"/>
+          <state_interface name="position">
+            <param name="initial_value">0.0</param>
+          </state_interface>
+        </joint>
+        <joint name="l_ank_roll">
+          <command_interface name="position"/>
+          <state_interface name="position">
+            <param name="initial_value">0.0</param>
+          </state_interface>
+        </joint>
+        <!-- Right Leg -->
+        <joint name="r_hip_yaw">
+          <command_interface name="position"/>
+          <state_interface name="position">
+            <param name="initial_value">0.0</param>
+          </state_interface>
+        </joint>
+        <joint name="r_hip_roll">
+          <command_interface name="position"/>
+          <state_interface name="position">
+            <param name="initial_value">0.0</param>
+          </state_interface>
+        </joint>
+        <joint name="r_hip_pitch">
+          <command_interface name="position"/>
+          <state_interface name="position">
+            <param name="initial_value">0.0</param>
+          </state_interface>
+        </joint>
+        <joint name="r_knee">
+          <command_interface name="position"/>
+          <state_interface name="position">
+            <param name="initial_value">0.0</param>
+          </state_interface>
+        </joint>
+        <joint name="r_ank_pitch">
+          <command_interface name="position"/>
+          <state_interface name="position">
+            <param name="initial_value">0.0</param>
+          </state_interface>
+        </joint>
+        <joint name="r_ank_roll">
+          <command_interface name="position"/>
+          <state_interface name="position">
+            <param name="initial_value">0.0</param>
+          </state_interface>
+        </joint>
+        <!-- Head -->
+        <joint name="head_pan">
+          <command_interface name="position"/>
+          <state_interface name="position">
+            <param name="initial_value">0.0</param>
+          </state_interface>
+        </joint>
+        <joint name="head_tilt">
+          <command_interface name="position"/>
+          <state_interface name="position">
+            <param name="initial_value">0.0</param>
+          </state_interface>
+        </joint>
+      </ros2_control>
+    </xacro:if>
+    <!-- ============================================================== -->
+    <!-- REAL HARDWARE: body system (22 DOF serial bus)                  -->
+    <!-- ============================================================== -->
+    <xacro:unless value="${use_gazebo}">
+      <ros2_control name="body_hardware" type="system">
+        <hardware>
           <plugin>rhphumanoid_hardware/RHPHumanoidSystemHardware</plugin>
           <param name="example_param_hw_start_duration_sec">0.0</param>
           <param name="example_param_hw_stop_duration_sec">2.0</param>
           <param name="example_param_hw_slowdown">10.0</param>
-        </xacro:unless>
-      </hardware>
-      <joint name="l_sho_pitch">
-        <command_interface name="position"/>
-        <state_interface name="position">
-          <param name="initial_value">0.15</param>
-        </state_interface>
-      </joint>
-      <joint name="l_sho_roll">
-        <command_interface name="position"/>
-        <state_interface name="position">
-          <param name="initial_value">-1.45</param>
-        </state_interface>
-      </joint>
-      <joint name="l_el">
-        <command_interface name="position"/>
-        <state_interface name="position">
-          <param name="initial_value">0.0</param>
-        </state_interface>
-      </joint>
-      <joint name="l_wst">
-        <command_interface name="position"/>
-        <state_interface name="position">
-          <param name="initial_value">-0.5</param>
-        </state_interface>
-      </joint>
-      <joint name="l_grp">
-        <command_interface name="position"/>
-        <state_interface name="position">
-          <param name="initial_value">0.0</param>
-        </state_interface>
-      </joint>
-      <joint name="r_sho_pitch">
-        <command_interface name="position"/>
-        <state_interface name="position">
-          <param name="initial_value">-0.15</param>
-        </state_interface>
-      </joint>
-      <joint name="r_sho_roll">
-        <command_interface name="position"/>
-        <state_interface name="position">
-          <param name="initial_value">1.45</param>
-        </state_interface>
-      </joint>
-      <joint name="r_el">
-        <command_interface name="position"/>
-        <state_interface name="position">
-          <param name="initial_value">0.0</param>
-        </state_interface>
-      </joint>
-      <joint name="r_wst">
-        <command_interface name="position"/>
-        <state_interface name="position">
-          <param name="initial_value">0.5</param>
-        </state_interface>
-      </joint>
-      <joint name="r_grp">
-        <command_interface name="position"/>
-        <state_interface name="position">
-          <param name="initial_value">0.0</param>
-        </state_interface>
-      </joint>
-      <joint name="l_hip_yaw">
-        <command_interface name="position"/>
-        <state_interface name="position">
-          <param name="initial_value">0.0</param>
-        </state_interface>
-      </joint>
-      <joint name="l_hip_roll">
-        <command_interface name="position"/>
-        <state_interface name="position">
-          <param name="initial_value">0.0</param>
-        </state_interface>
-      </joint>
-      <joint name="l_hip_pitch">
-        <command_interface name="position"/>
-        <state_interface name="position">
-          <param name="initial_value">0.0</param>
-        </state_interface>
-      </joint>
-      <joint name="l_knee">
-        <command_interface name="position"/>
-        <state_interface name="position">
-          <param name="initial_value">0.0</param>
-        </state_interface>
-      </joint>
-      <joint name="l_ank_pitch">
-        <command_interface name="position"/>
-        <state_interface name="position">
-          <param name="initial_value">0.0</param>
-        </state_interface>
-      </joint>
-      <joint name="l_ank_roll">
-        <command_interface name="position"/>
-        <state_interface name="position">
-          <param name="initial_value">0.0</param>
-        </state_interface>
-      </joint>
-      <joint name="r_hip_yaw">
-        <command_interface name="position"/>
-        <state_interface name="position">
-          <param name="initial_value">0.0</param>
-        </state_interface>
-      </joint>
-      <joint name="r_hip_roll">
-        <command_interface name="position"/>
-        <state_interface name="position">
-          <param name="initial_value">0.0</param>
-        </state_interface>
-      </joint>
-      <joint name="r_hip_pitch">
-        <command_interface name="position"/>
-        <state_interface name="position">
-          <param name="initial_value">0.0</param>
-        </state_interface>
-      </joint>
-      <joint name="r_knee">
-        <command_interface name="position"/>
-        <state_interface name="position">
-          <param name="initial_value">0.0</param>
-        </state_interface>
-      </joint>
-      <joint name="r_ank_pitch">
-        <command_interface name="position"/>
-        <state_interface name="position">
-          <param name="initial_value">0.0</param>
-        </state_interface>
-      </joint>
-      <joint name="r_ank_roll">
-        <command_interface name="position"/>
-        <state_interface name="position">
-          <param name="initial_value">0.0</param>
-        </state_interface>
-      </joint>
-      <joint name="head_pan">
-        <command_interface name="position"/>
-        <state_interface name="position">
-          <param name="initial_value">0.0</param>
-        </state_interface>
-      </joint>
-      <joint name="head_tilt">
-        <command_interface name="position"/>
-        <state_interface name="position">
-          <param name="initial_value">0.0</param>
-        </state_interface>
-      </joint>
-    </ros2_control>
+        </hardware>
+        <!-- Left Arm -->
+        <joint name="l_sho_pitch">
+          <command_interface name="position"/>
+          <state_interface name="position">
+            <param name="initial_value">0.15</param>
+          </state_interface>
+        </joint>
+        <joint name="l_sho_roll">
+          <command_interface name="position"/>
+          <state_interface name="position">
+            <param name="initial_value">-1.45</param>
+          </state_interface>
+        </joint>
+        <joint name="l_el">
+          <command_interface name="position"/>
+          <state_interface name="position">
+            <param name="initial_value">0.0</param>
+          </state_interface>
+        </joint>
+        <joint name="l_wst">
+          <command_interface name="position"/>
+          <state_interface name="position">
+            <param name="initial_value">-0.5</param>
+          </state_interface>
+        </joint>
+        <joint name="l_grp">
+          <command_interface name="position"/>
+          <state_interface name="position">
+            <param name="initial_value">0.0</param>
+          </state_interface>
+        </joint>
+        <!-- Right Arm -->
+        <joint name="r_sho_pitch">
+          <command_interface name="position"/>
+          <state_interface name="position">
+            <param name="initial_value">-0.15</param>
+          </state_interface>
+        </joint>
+        <joint name="r_sho_roll">
+          <command_interface name="position"/>
+          <state_interface name="position">
+            <param name="initial_value">1.45</param>
+          </state_interface>
+        </joint>
+        <joint name="r_el">
+          <command_interface name="position"/>
+          <state_interface name="position">
+            <param name="initial_value">0.0</param>
+          </state_interface>
+        </joint>
+        <joint name="r_wst">
+          <command_interface name="position"/>
+          <state_interface name="position">
+            <param name="initial_value">0.5</param>
+          </state_interface>
+        </joint>
+        <joint name="r_grp">
+          <command_interface name="position"/>
+          <state_interface name="position">
+            <param name="initial_value">0.0</param>
+          </state_interface>
+        </joint>
+        <!-- Left Leg -->
+        <joint name="l_hip_yaw">
+          <command_interface name="position"/>
+          <state_interface name="position">
+            <param name="initial_value">0.0</param>
+          </state_interface>
+        </joint>
+        <joint name="l_hip_roll">
+          <command_interface name="position"/>
+          <state_interface name="position">
+            <param name="initial_value">0.0</param>
+          </state_interface>
+        </joint>
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
File: rhphumanoid_description/urdf/rhphumanoid.structure.head.xacro (robot description, xacro)
@@ -60,5 +60,5 @@
   </link>
   <!-- camera joint -->
-  <!-- <joint name="cam" type="fixed">
+  <joint name="cam" type="fixed">
     <origin xyz="0.01425 -0.019 0.04975" rpy="${-pi*0.5} 0 ${-pi*0.5}"/>
     <parent link="head_tilt_link"/>
@@ -69,11 +69,11 @@
     <parent link="head_tilt_link"/>
     <child link="cam_gazebo_link"/>
-  </joint> -->
+  </joint>
   <!-- camera link -->
-  <!-- <link name="cam_link">
-  </link> -->
+  <link name="cam_link">
+  </link>
   <!-- camera link -->
-  <!-- <link name="cam_gazebo_link">
-  </link> -->
+  <link name="cam_gazebo_link">
+  </link>
   </xacro:macro>
 </robot>
