Commit message: [Modify] Head Only

File: rhphumanoid_description/ros2_control/rhphumanoid.ros2_control.xacro (robot description, xacro)
@@ -1,5 +1,5 @@
 <?xml version="1.0"?>
 <robot xmlns:xacro="http://www.ros.org/wiki/xacro">
-  <xacro:macro name="rhphumanoid_ros2_control" params="name use_gazebo:=^|false">
+  <xacro:macro name="rhphumanoid_ros2_control" params="name use_gazebo:=^|false head_only:=false">
     <!-- ============================================================== -->
     <!-- GAZEBO SIMULATION: single system with all 24 joints            -->
@@ -165,4 +165,5 @@
     <!-- ============================================================== -->
     <xacro:unless value="${use_gazebo}">
+      <xacro:unless value="${head_only}">
       <ros2_control name="body_hardware" type="system">
         <hardware>
@@ -309,4 +310,5 @@
         </joint>
       </ros2_control>
+      </xacro:unless>
       <!-- ============================================================== -->
       <!-- REAL HARDWARE: head system (2 DOF PWM servos)                   -->

File: rhphumanoid_description/urdf/rhphumanoid.urdf.xacro (robot description, xacro)
@@ -2,4 +2,5 @@
 <robot xmlns:xacro="http://ros.org/wiki/xacro" name="rhphumanoid">
   <xacro:arg name="use_gazebo" default="false" />
+  <xacro:arg name="head_only" default="false" />
   <xacro:include filename="$(find rhphumanoid_description)/urdf/rhphumanoid.visuals.xacro" />
   <xacro:include filename="$(find rhphumanoid_description)/urdf/rhphumanoid.inertia.xacro" />
@@ -38,5 +39,5 @@
   <xacro:rhphumanoid_r_leg parent="body_link" />
   <xacro:rhphumanoid_l_leg parent="body_link" />
-  <xacro:rhphumanoid_ros2_control name="RHPHumanoid" use_gazebo="$(arg use_gazebo)" />
+  <xacro:rhphumanoid_ros2_control name="RHPHumanoid" use_gazebo="$(arg use_gazebo)" head_only="$(arg head_only)" />
   <!-- head links -->
   <xacro:rhphumanoid_head parent="body_link" />
